Commit message: Updated URDF with Zed-M and YDLidar T-Mini plus

File: src/robot_description/urdf/sora.urdf (robot description, URDF)
Before this commit: robot sora, 7 links, 6 joints
Links:
- added link base_link
- added link laser_frame
- added link zed_camera_center
- link baseplate: mass 7.5335 -> 5.17808; geometry collision mesh filename=package://Sora/assets/baseplate.stl; collision mesh filename=package://Sora/assets/defuser.stl
- link liftingmechanism: geometry collision mesh filename=package://Sora/assets/liftingplatform1.stl; collision mesh filename=package://Sora/assets/liftingplatform2.stl
- link liftingmechanism_2: geometry collision mesh filename=package://Sora/assets/liftingplatform1.stl; collision mesh filename=package://Sora/assets/liftingplatform2.stl
- link mecanum_wheel___left: geometry collision mesh filename=package://Sora/assets/rim_inside__2.stl; collision mesh filename=package://Sora/assets/rim_outside__2.stl
- link mecanum_wheel___left_2: geometry collision mesh filename=package://Sora/assets/rim_inside__2.stl; collision mesh filename=package://Sora/assets/rim_outside__2.stl
- link mecanum_wheel___right: geometry collision mesh filename=package://Sora/assets/rim_inside.stl; collision mesh filename=package://Sora/assets/rim_outside.stl
- link mecanum_wheel___right_2: geometry collision mesh filename=package://Sora/assets/rim_inside.stl; collision mesh filename=package://Sora/assets/rim_outside.stl
Joints:
- added joint base_link_to_baseplate: type fixed, parent base_link, child baseplate, origin xyz=0 0 0 rpy=0 0 0
- added joint base_link_to_laser: type fixed, parent base_link, child laser_frame, origin xyz=-0.135 0 0.115 rpy=0 0 0
- added joint base_link_to_zed: type fixed, parent base_link, child zed_camera_center, origin xyz=-0.160  0  0.069 rpy=0 0 0
- joint Lift_Left: limit lower=0 upper=0.022 effort=10 velocity=10 -> lower=0 upper=0.0195 effort=10 velocity=10; origin xyz=-0.015775 -0.073425 0.104 rpy=0 0 0 -> xyz=-0.015775 -0.073425 0.1015 rpy=0 0 0
- joint Lift_Right: limit lower=0 upper=0.022 effort=10 velocity=10 -> lower=0 upper=0.0195 effort=10 velocity=10; origin xyz=-0.015775 0.073425 0.104 rpy=0 0 0 -> xyz=-0.015775 0.073425 0.1015 rpy=0 0 0
- joint Wheel_BL: limit (none) -> lower=-3.1415927 upper=3.1415927 effort=10 velocity=10; origin xyz=0.3175 -0.14 0.024 rpy=1.5708 0 3.14159 -> xyz=0.3175 -0.135 0.024 rpy=1.5708 0 3.14159; type continuous -> revolute
- joint Wheel_BR: limit (none) -> lower=-3.1415927 upper=3.1415927 effort=10 velocity=10; origin xyz=0.3175 0.14 0.024 rpy=-1.5708 0 3.14159 -> xyz=0.3175 0.135 0.024 rpy=-1.5708 0 3.14159; type continuous -> revolute
- joint Wheel_FL: limit (none) -> lower=-3.1415927 upper=3.1415927 effort=10 velocity=10; origin xyz=-0.0925 -0.14 0.024 rpy=-1.5708 0 0 -> xyz=-0.0925 -0.135 0.024 rpy=-1.5708 0 0; type continuous -> revolute
- joint Wheel_FR: limit (none) -> lower=-3.1415927 upper=3.1415927 effort=10 velocity=10; origin xyz=-0.0925 0.14 0.024 rpy=1.5708 0 0 -> xyz=-0.0925 0.135 0.024 rpy=1.5708 0 0; type continuous -> revolute

Commit message: URDF changes for assets

File: src/robot_description/urdf/sora.urdf (robot description, URDF)
Before this commit: robot sora, 10 links, 9 joints
Links:
- link baseplate: geometry collision mesh filename=package://robot_description/assets/baseplate.stl; collision mesh filename=package://robot_description/assets/defuser.stl
- link liftingmechanism: geometry collision mesh filename=package://robot_description/assets/liftingplatform1.stl; collision mesh filename=package://robot_description/assets/liftingplatform2.stl
- link liftingmechanism_2: geometry collision mesh filename=package://robot_description/assets/liftingplatform1.stl; collision mesh filename=package://robot_description/assets/liftingplatform2.stl
- link mecanum_wheel___left: geometry collision mesh filename=package://robot_description/assets/rim_inside__2.stl; collision mesh filename=package://robot_description/assets/rim_outside__2.stl
- link mecanum_wheel___left_2: geometry collision mesh filename=package://robot_description/assets/rim_inside__2.stl; collision mesh filename=package://robot_description/assets/rim_outside__2.stl
- link mecanum_wheel___right: geometry collision mesh filename=package://robot_description/assets/rim_inside.stl; collision mesh filename=package://robot_description/assets/rim_outside.stl
- link mecanum_wheel___right_2: geometry collision mesh filename=package://robot_description/assets/rim_inside.stl; collision mesh filename=package://robot_description/assets/rim_outside.stl

Commit message: URDF orientation fix

File: src/robot_description/urdf/sora.urdf (robot description, URDF)
Before this commit: robot sora, 10 links, 9 joints
Links:
- added link zedm_camera_center
Joints:
- added joint zed_camera_center_to_zedm_camera_center: type fixed, parent zed_camera_center, child zedm_camera_center, origin xyz=0 0 0 rpy=0 0 0
- joint base_link_to_baseplate: origin xyz=0 0 0 rpy=0 0 0 -> xyz=0 0 0 rpy=0 0 3.141592653589793
- joint base_link_to_laser: origin xyz=-0.135 0 0.115 rpy=0 0 0 -> xyz=0.135 0 0.115 rpy=0 0 0
- joint base_link_to_zed: origin xyz=-0.160  0  0.069 rpy=0 0 0 -> xyz=0.160 0 0.069 rpy=0 0 0

Commit message: odom and mapping changes

File: src/robot_description/urdf/sora.urdf (robot description, URDF)
Before this commit: robot sora, 11 links, 10 joints
Links:
- removed link zedm_camera_center
Joints:
- removed joint zed_camera_center_to_zedm_camera_center
- joint base_link_to_laser: origin xyz=0.135 0 0.115 rpy=0 0 0 -> xyz=0.135 0 0.115 rpy=0 0 3.141592653589793

Commit message: saving maps

File: src/robot_description/urdf/sora.urdf (robot description, URDF)
Before this commit: robot sora, 10 links, 9 joints
Joints:
- joint base_link_to_laser: origin xyz=0.135 0 0.115 rpy=0 0 3.141592653589793 -> xyz=0.135 0 0.115 rpy=0 0 0

Commit message: urdf change

File: src/robot_description/urdf/sora.urdf (robot description, URDF)
Before this commit: robot sora, 10 links, 9 joints
Links:
- removed link zed_camera_center
- added link zedm_camera_center
Joints:
- joint base_link_to_zed: child zed_camera_center -> zedm_camera_center

Commit message: urdf changes

File: src/robot_description/urdf/sora.urdf (robot description, URDF)
Before this commit: robot sora, 10 links, 9 joints
Links:
- removed link zedm_camera_center
- added link zed_mount
Joints:
- removed joint base_link_to_zed
- added joint base_link_to_zed_mount: type fixed, parent base_link, child zed_mount, origin xyz=0.160 0 0.069 rpy=0 0 0
